File: hardware/ring/R30-OLED-NONE-NONE/kicad/sheets/usb_and_service.kicad_sch (KiCad schematic)
At the start: 0 parts

Commit message: feat(hardware): scaffold 30deg optical ring sensor/click and usb interfaces for accessibility pointing, ~$9 ring BOM
Other:
- note added: "USB and service interface scaffold: VBUS entry, CC sink-attach, ESD protection, and native USB data nets are locked here before the USB-C receptacle, ESD array, and service pads land."
Changed lines of the file:
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@@
   (generator_version "0.1")
   (paper "A4")
+  (text "USB and service interface scaffold: VBUS entry, CC sink-attach, ESD protection, and native USB data nets are locked here before the USB-C receptacle, ESD array, and service pads land."
+    (at 20.32 20.32 0)
+    (effects (font (size 1.27 1.27)))
+  )
+  (hierarchical_label "VBUS_5V"
+    (shape output)
+    (at 187.96 38.1 180)
+    (effects (font (size 1.27 1.27)))
+  )
+  (hierarchical_label "USB_D+"
+    (shape bidirectional)
+    (at 187.96 45.72 180)
+    (effects (font (size 1.27 1.27)))
+  )
+  (hierarchical_label "USB_D-"
+    (shape bidirectional)
+    (at 187.96 53.34 180)
+    (effects (font (size 1.27 1.27)))
+  )
   (sheet_instances
     (path "/" (page "1"))
