File: hardware/shared/USB-HUB/kicad/sheets/usb_and_power.kicad_sch (KiCad schematic)
At the start: 7 parts, among them J1 SOFNG USB-05, U2 RT9080-33GJ5

Commit message: fix(usb-hub): clean native-usb dongle drc parity
Direct-plug native USB hub dongle for accessibility pointing and OCR composition; no sensing mechanism change; BOM intent remains ~-6.
Parts:
- added C1B: 100nF, Capacitor_SMD:C_0402_1005Metric, symbol Device:C
Connections:
- net GND: now also J1.SH1 (SHIELD), J1.SH2 (SHIELD), C1B.2
- net VREG_3V3: now also C1B.1
Changed lines of the file:
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@@
     (effects (font (size 1.27 1.27)) (justify left bottom))
   )
-  (label "GND"
+  (hierarchical_label "GND"
+    (shape passive)
     (at 160.02 48.26 0)
     (effects (font (size 1.27 1.27)) (justify left bottom))
@@
   (wire
     (pts
+      (xy 48.26 60.96)
+      (xy 60.96 60.96)
+    )
+    (stroke (width 0) (type default) (color 0 0 0 0))
+  )
+  (wire
+    (pts
+      (xy 48.26 63.5)
+      (xy 60.96 63.5)
+    )
+    (stroke (width 0) (type default) (color 0 0 0 0))
+  )
+  (label "GND"
+    (at 60.96 60.96 0)
+    (effects (font (size 1.27 1.27)) (justify left bottom))
+  )
+  (label "GND"
+    (at 60.96 63.5 0)
+    (effects (font (size 1.27 1.27)) (justify left bottom))
+  )
+  (wire
+    (pts
       (xy 81.28 50.8)
       (xy 73.66 50.8)
@@
     (pin "3")
     (pin "4")
+    (pin "SH1")
+    (pin "SH2")
     (instances
       (project "usb_hub"
@@
         )
       )
+    )
+  )
+  (label "VREG_3V3"
+    (at 187.96 52.07 0)
+    (effects (font (size 1.27 1.27)) (justify left bottom))
+  )
+  (label "GND"
+    (at 187.96 59.69 0)
+    (effects (font (size 1.27 1.27)) (justify left bottom))
+  )
+  (wire
+    (pts
+      (xy 180.34 52.07)
+      (xy 187.96 52.07)
+    )
+    (stroke (width 0) (type default) (color 0 0 0 0))
+  )
+  (wire
+    (pts
+      (xy 180.34 59.69)
+      (xy 187.96 59.69)
+    )
+    (stroke (width 0) (type default) (color 0 0 0 0))
+  )
+  (symbol (lib_id "Device:C") (at 180.34 55.88 0) (unit 1)
+    (in_bom yes) (on_board yes) (dnp no) (fields_autoplaced)
+    (property "Reference" "C1B" (at 175.26 49.53 0)
+      (effects (font (size 1.27 1.27)) (justify left))
+    )
+    (property "Value" "100nF" (at 175.26 52.07 0)
+      (effects (font (size 1.27 1.27)) (justify left))
+    )
+    (property "Footprint" "Capacitor_SMD:C_0402_1005Metric" (at 180.34 45.72 0)
+      (effects (font (size 1.27 1.27)) hide)
+    )
+    (property "Datasheet" "" (at 180.34 43.18 0)
+      (effects (font (size 1.27 1.27)) hide)
+    )
+    (pin "1")
+    (pin "2")
+    (instances
+      (project "usb_hub"
+        (path "/"
+          (reference "C1B") (unit 1)
+        )
+      )

Commit message: fix(usb-hub): pin local first-board footprints
Design disclosure: sensing mechanism none; form factor stepped USB-A direct-plug USB-HUB dongle; intended use offline BLE HID composition and service access for accessibility; BOM estimate ~$5-6 packet target.

Move first-board commodity/support footprints into the source-controlled PowerFinger_USB library and update the packet verification story to all-severity PCB DRC clean.
Parts:
- C1B: footprint Capacitor_SMD:C_0402_1005Metric -> PowerFinger_USB:C_0402_1005Metric_FirstBoard
- C2, C3: footprint Capacitor_SMD:C_0603_1608Metric -> PowerFinger_USB:C_0603_1608Metric_FirstBoard
- D1: footprint Package_TO_SOT_SMD:SOT-23-6 -> PowerFinger_USB:SOT-23-6_FirstBoard
- R1A, R1B: footprint Resistor_SMD:R_0402_1005Metric -> PowerFinger_USB:R_0402_1005Metric_FirstBoard
- U2: footprint Package_TO_SOT_SMD:SOT-23-5 -> PowerFinger_USB:SOT-23-5_FirstBoard
Changed lines of the file:
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@@
       (effects (font (size 1.27 1.27)) (justify left))
     )
-    (property "Footprint" "Package_TO_SOT_SMD:SOT-23-6" (at 88.9 33.02 0)
+    (property "Footprint" "PowerFinger_USB:SOT-23-6_FirstBoard" (at 88.9 33.02 0)
       (effects (font (size 1.27 1.27)) hide)
     )
@@
       (effects (font (size 1.27 1.27)) (justify left))
     )
-    (property "Footprint" "Package_TO_SOT_SMD:SOT-23-5" (at 152.4 20.32 0)
+    (property "Footprint" "PowerFinger_USB:SOT-23-5_FirstBoard" (at 152.4 20.32 0)
       (effects (font (size 1.27 1.27)) hide)
     )
@@
       (effects (font (size 1.27 1.27)))
     )
-    (property "Footprint" "Resistor_SMD:R_0402_1005Metric" (at 142.24 48.26 0)
+    (property "Footprint" "PowerFinger_USB:R_0402_1005Metric_FirstBoard" (at 142.24 48.26 0)
       (effects (font (size 1.27 1.27)) hide)
     )
@@
       (effects (font (size 1.27 1.27)))
     )
-    (property "Footprint" "Resistor_SMD:R_0402_1005Metric" (at 142.24 40.64 0)
+    (property "Footprint" "PowerFinger_USB:R_0402_1005Metric_FirstBoard" (at 142.24 40.64 0)
       (effects (font (size 1.27 1.27)) hide)
     )
@@
       (effects (font (size 1.27 1.27)) (justify left))
     )
-    (property "Footprint" "Capacitor_SMD:C_0603_1608Metric" (at 119.38 29.21 0)
+    (property "Footprint" "PowerFinger_USB:C_0603_1608Metric_FirstBoard" (at 119.38 29.21 0)
       (effects (font (size 1.27 1.27)) hide)
     )
@@
       (effects (font (size 1.27 1.27)) (justify left))
     )
-    (property "Footprint" "Capacitor_SMD:C_0603_1608Metric" (at 170.18 20.32 0)
+    (property "Footprint" "PowerFinger_USB:C_0603_1608Metric_FirstBoard" (at 170.18 20.32 0)
       (effects (font (size 1.27 1.27)) hide)
     )
@@
       (effects (font (size 1.27 1.27)) (justify left))
     )
-    (property "Footprint" "Capacitor_SMD:C_0402_1005Metric" (at 180.34 45.72 0)
+    (property "Footprint" "PowerFinger_USB:C_0402_1005Metric_FirstBoard" (at 180.34 45.72 0)
       (effects (font (size 1.27 1.27)) hide)
     )
