File: hardware/shared/USB-HUB/kicad/sheets/usb_and_power.kicad_sch (KiCad schematic)
At the start: 8 parts, among them J1 SOFNG USB-05, U2 RT9080-33GJ5

Commit message: fix(usb-hub): close kicad erc snapshot
Changed lines of the file:
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@@
-  (wire
-    (pts
-      (xy 60.96 40.64)
-      (xy 68.58 40.64)
-    )
-    (stroke (width 0) (type default) (color 0 0 0 0))
-  )
   (wire
     (pts
@@
       (xy 48.26 55.88)
       (xy 60.96 55.88)
-    )
-    (stroke (width 0) (type default) (color 0 0 0 0))
-  )
-  (wire
-    (pts
-      (xy 60.96 55.88)
-      (xy 68.58 55.88)
     )
     (stroke (width 0) (type default) (color 0 0 0 0))
@@
     (stroke (width 0) (type default) (color 0 0 0 0))
   )
-  (symbol (lib_id "power:PWR_FLAG") (at 68.58 40.64 0) (unit 1)
-    (in_bom no) (on_board no) (dnp no)
-    (property "Reference" "#FLG0101" (at 68.58 38.735 0)
-      (effects (font (size 1.27 1.27)) hide)
-    )
-    (property "Value" "PWR_FLAG" (at 68.58 36.83 0)
-      (effects (font (size 1.27 1.27)))
-    )
-    (pin "1")
-    (instances
-      (project "usb_hub"
-        (path "/"
-          (reference "#FLG0101") (unit 1)
-        )
-      )
-    )
-  )
-  (symbol (lib_id "power:PWR_FLAG") (at 68.58 55.88 0) (unit 1)
-    (in_bom no) (on_board no) (dnp no)
-    (property "Reference" "#FLG0102" (at 68.58 53.975 0)
-      (effects (font (size 1.27 1.27)) hide)
-    )
-    (property "Value" "PWR_FLAG" (at 68.58 52.07 0)
-      (effects (font (size 1.27 1.27)))
-    )
-    (pin "1")
-    (instances
-      (project "usb_hub"
-        (path "/"
-          (reference "#FLG0102") (unit 1)
-        )
-      )
-    )
-  )
   (symbol (lib_id "PowerFinger:USB_A_Plug_Male") (at 40.64 48.26 0) (unit 1)
